Commit message: TBD simulating ensenso in gazebo

File: godel_robots/blending_end_effector/urdf/blending_eff_macro.xacro (robot description, xacro)
@@ -132,6 +132,36 @@
     </joint>
     <!--Frames related to the motion of the camera-->
-    <link name="${prefix}ensenso_sensor_optical_frame"/>
-    <link name="${prefix}kinect2_move_frame"/>
+    <link name="${prefix}ensenso_sensor_optical_frame">
+    <inertial>
+      <mass value="0.001" />
+      <origin xyz="0 0 0" />
+      <inertia ixx="0.0001" ixy="0.0" ixz="0.0"
+               iyy="0.0001" iyz="0.0"
+               izz="0.0001" />
+    </inertial>
+    </link>
+    <link name="${prefix}kinect2_move_frame">
+    <inertial>
+      <mass value="0.001" />
+      <origin xyz="0 0 0" />
+      <inertia ixx="0.0001" ixy="0.0" ixz="0.0"
+               iyy="0.0001" iyz="0.0"
+               izz="0.0001" />
+    </inertial>
+    </link>
+    <link name="${prefix}ensenso_frame">
+        <inertial>
+          <mass value="0.001" />
+          <origin xyz="0 0 0" />
+          <inertia ixx="0.0001" ixy="0.0" ixz="0.0"
+                   iyy="0.0001" iyz="0.0"
+                   izz="0.0001" />
+        </inertial>
+    </link>
+    <joint name="${prefix}ensenso_joint" type="fixed">
+        <parent link="${prefix}ensenso_sensor_optical_frame"/>
+        <child link="${prefix}ensenso_frame"/>
+        <origin xyz="0 0 0" rpy="-1.57 0 -1.57"/>
+    </joint>
     <joint name="${prefix}bracket_to_ensenso_sof" type="fixed">
         <parent link="${prefix}bracket"/>
@@ -144,4 +174,40 @@
       <origin rpy="0 -${half_pi} 0"/>
     </joint>
+    <gazebo reference="ensenso_sensor_optical_frame">
+      <sensor type="depth" name="ensenso">
+        <always_on>true</always_on>
+        <update_rate>20.0</update_rate>
+        <camera>
+          <horizontal_fov>${60.0*M_PI/180.0}</horizontal_fov>
+          <image>
+            <format>B8G8R8</format>
+            <width>640</width>
+            <height>480</height>
+          </image>
+          <clip>
+            <near>0.05</near>
+            <far>8.0</far>
+          </clip>
+        </camera>
+        <plugin name="kinect_camera_controller" filename="libgazebo_ros_openni_kinect.so">
+          <cameraName>ensenso</cameraName>
+          <alwaysOn>true</alwaysOn>
+          <updateRate>10</updateRate>
+          <imageTopicName>rgb/image_raw</imageTopicName>
+          <depthImageTopicName>depth/image_raw</depthImageTopicName>
+          <pointCloudTopicName>depth/points</pointCloudTopicName>
+          <cameraInfoTopicName>rgb/camera_info</cameraInfoTopicName>
+          <depthImageCameraInfoTopicName>depth/camera_info</depthImageCameraInfoTopicName>
+          <frameName>ensenso_frame</frameName>
+          <baseline>0.1</baseline>
+          <distortion_k1>0.0</distortion_k1>
+          <distortion_k2>0.0</distortion_k2>
+          <distortion_k3>0.0</distortion_k3>
+          <distortion_t1>0.0</distortion_t1>
+          <distortion_t2>0.0</distortion_t2>
+          <pointCloudCutoff>0.4</pointCloudCutoff>
+        </plugin>
+      </sensor>
+    </gazebo>
   </xacro:macro>
 </robot>

File: godel_robots/denso/godel_denso_support/urdf/denso_demo_description.urdf.xacro (robot description, xacro)
@@ -22,8 +22,8 @@
 	</joint>
 	<!--xacro:if value="${sim}"-->
-	  <xacro:sensor_kinect parent="world_frame">
+          <xacro:sensor_kinect parent="world_frame">
 	    <origin xyz="0.27 0.9 1.23" rpy="0 ${pi/2 - 15 * pi/180} ${-pi/2}"/>
 	  </xacro:sensor_kinect>
-	<!--/xacro:if-->
+        <!--/xacro:if-->
 	<!-- include camera -->
 	<!--xacro:unless value="${sim}">

Commit message: Added ensenso according to kinect

File: godel_robots/blending_end_effector/urdf/blending_eff_macro.xacro (robot description, xacro)
@@ -150,4 +150,18 @@
     </inertial>
     </link>
+    <link name="${prefix}ensenso_depth_optical_frame">
+        <inertial>
+          <mass value="0.001" />
+          <origin xyz="0 0 0" />
+          <inertia ixx="0.0001" ixy="0.0" ixz="0.0"
+                   iyy="0.0001" iyz="0.0"
+                   izz="0.0001" />
+        </inertial>
+    </link>
+    <joint name="${prefix}ensenso_optical_joint" type="fixed">
+        <parent link="${prefix}ensenso_sensor_optical_frame"/>
+        <child link="${prefix}ensenso_depth_optical_frame"/>
+        <origin xyz="0 0 0" rpy="-1.57 0 -1.57"/>
+    </joint>
     <link name="${prefix}ensenso_frame">
         <inertial>
@@ -160,5 +174,5 @@
     </link>
     <joint name="${prefix}ensenso_joint" type="fixed">
-        <parent link="${prefix}ensenso_sensor_optical_frame"/>
+        <parent link="${prefix}ensenso_depth_optical_frame"/>
         <child link="${prefix}ensenso_frame"/>
         <origin xyz="0 0 0" rpy="-1.57 0 -1.57"/>
@@ -199,5 +213,5 @@
           <cameraInfoTopicName>rgb/camera_info</cameraInfoTopicName>
           <depthImageCameraInfoTopicName>depth/camera_info</depthImageCameraInfoTopicName>
-          <frameName>ensenso_frame</frameName>
+          <frameName>ensenso_depth_optical_frame</frameName>
           <baseline>0.1</baseline>
           <distortion_k1>0.0</distortion_k1>

Commit message: TBD executing blending trajectories

File: godel_robots/blending_end_effector/urdf/blending_eff_macro.xacro (robot description, xacro)
@@ -65,6 +65,8 @@
     <link name="${prefix}blending_tool">
         <visual>
+            <!--origin xyz="0 0 0.1" rpy="0 0 0"/-->
             <geometry>
                 <mesh filename="package://blending_end_effector/meshes/visual/Blending_Tool.STL"/>
+                <!--cylinder length="0.05" radius="0.01"/-->
             </geometry>
             <material name="red">
@@ -162,5 +164,5 @@
         <parent link="${prefix}ensenso_sensor_optical_frame"/>
         <child link="${prefix}ensenso_depth_optical_frame"/>
-        <origin xyz="0 0 0" rpy="-1.57 0 -1.57"/>
+        <origin xyz="0 0 0" rpy="0 0 -3.142"/>
     </joint>
     <link name="${prefix}ensenso_frame">
@@ -176,5 +178,5 @@
         <parent link="${prefix}ensenso_depth_optical_frame"/>
         <child link="${prefix}ensenso_frame"/>
-        <origin xyz="0 0 0" rpy="-1.57 0 -1.57"/>
+        <origin xyz="0 0 0" rpy="1.57 -1.57 0"/>
     </joint>
     <joint name="${prefix}bracket_to_ensenso_sof" type="fixed">
@@ -188,10 +190,10 @@
       <origin rpy="0 -${half_pi} 0"/>
     </joint>
-    <gazebo reference="ensenso_sensor_optical_frame">
+    <gazebo reference="ensenso_frame">
       <sensor type="depth" name="ensenso">
         <always_on>true</always_on>
         <update_rate>20.0</update_rate>
         <camera>
-          <horizontal_fov>${60.0*M_PI/180.0}</horizontal_fov>
+          <horizontal_fov>${60.0*3.142/180.0}</horizontal_fov>
           <image>
             <format>B8G8R8</format>
@@ -200,5 +202,5 @@
           </image>
           <clip>
-            <near>0.05</near>
+            <near>0.001</near>
             <far>8.0</far>
           </clip>
@@ -220,5 +222,5 @@
           <distortion_t1>0.0</distortion_t1>
           <distortion_t2>0.0</distortion_t2>
-          <pointCloudCutoff>0.4</pointCloudCutoff>
+          <pointCloudCutoff>0.1</pointCloudCutoff>
         </plugin>
       </sensor>

File: godel_robots/denso/godel_denso_support/urdf/denso_demo_description.urdf.xacro (robot description, xacro)
@@ -6,32 +6,38 @@
   <xacro:include filename="$(find blending_end_effector)/urdf/blending_eff_macro.xacro"/>
   <!--xacro:property name="sim" value="$(arg sim)"/-->
-	<link name="world_frame"/>
-	<!-- include platform -->
-	<xacro:table prefix="" parent="world_frame">
-  	  <origin xyz="-0.24 -0.78 -0.75" rpy="0 0 0"/>
-	</xacro:table>
-  	<!-- arm -->
-	<xacro:vs087 prefix="" parent="world_frame">
+    <link name="world_frame"/>
+    <!-- include platform -->
+    <xacro:table prefix="" parent="world_frame">
+      <origin xyz="-0.24 -0.78 -0.75" rpy="0 0 0"/>
+    </xacro:table>
+    <!-- arm -->
+    <xacro:vs087 prefix="" parent="world_frame">
  	  <origin xyz="0 0 0" rpy="0 0 0" />
     </xacro:vs087>
     <xacro:blending_eff_definition prefix=""/>
+    <link name="tool0"/>
+    <joint name="tool0_joint" type="fixed">
+        <origin xyz="0 0 0" rpy="0 -${half_pi} 0" />
+        <parent link="link_6" />
+        <child link="tool0" />
+    </joint>
     <joint name="eff_joint" type="fixed">
-		<origin xyz="0 0 0" rpy="0 0 0" />
-		<parent link="link_6" />
+        <origin xyz="0 0 0" rpy="0 0 ${half_pi}" />
+        <parent link="tool0" />
         <child link="eff_frame" />
-	</joint>
-	<!--xacro:if value="${sim}"-->
-          <xacro:sensor_kinect parent="world_frame">
-	    <origin xyz="0.27 0.9 1.23" rpy="0 ${pi/2 - 15 * pi/180} ${-pi/2}"/>
-	  </xacro:sensor_kinect>
-        <!--/xacro:if-->
-	<!-- include camera -->
-	<!--xacro:unless value="${sim}">
-	  <link name="camera_link"/>
-	  <joint name="camera_joint" type="fixed">
-		<parent link="world"/>
-		<child link="camera_link"/>
-		<origin xyz="0.27 0.9 1.23" rpy="0 ${pi/2 - 15 * pi/180} ${-pi/2}"/>
-	  </joint>
-	</xacro:unless-->
+    </joint>
+    <!--xacro:if value="${sim}"-->
+      <xacro:sensor_kinect parent="world_frame">
+        <origin xyz="0.27 0.9 1.23" rpy="0 ${pi/2 - 15 * pi/180} ${-pi/2}"/>
+      </xacro:sensor_kinect>
+    <!--/xacro:if-->
+    <!-- include camera -->
+    <!--xacro:unless value="${sim}">
+      <link name="camera_link"/>
+      <joint name="camera_joint" type="fixed">
+            <parent link="world"/>
+            <child link="camera_link"/>
+            <origin xyz="0.27 0.9 1.23" rpy="0 ${pi/2 - 15 * pi/180} ${-pi/2}"/>
+      </joint>
+    </xacro:unless-->
 </robot>

Commit message: Scan n plan works with track_ik. TDB: blend exec

File: godel_robots/blending_end_effector/urdf/blending_eff_macro.xacro (robot description, xacro)
@@ -65,8 +65,8 @@
     <link name="${prefix}blending_tool">
         <visual>
-            <!--origin xyz="0 0 0.1" rpy="0 0 0"/-->
+            <origin xyz="0 0 0.1" rpy="0 0 0"/>
             <geometry>
-                <mesh filename="package://blending_end_effector/meshes/visual/Blending_Tool.STL"/>
-                <!--cylinder length="0.05" radius="0.01"/-->
+                <!--mesh filename="package://blending_end_effector/meshes/visual/Blending_Tool.STL"/-->
+                <cylinder length="0.2" radius="0.01"/>
             </geometry>
             <material name="red">
@@ -78,4 +78,9 @@
         <parent link="${prefix}bracket"/>
         <child link="${prefix}blending_tool"/>
+    </joint>
+    <joint name="${prefix}chuck_to_blend_tcp_frame" type="fixed">
+        <parent link="${prefix}blending_tool"/>
+        <child link="${prefix}tcp_frame"/>
+        <origin xyz="0 0 0.2" rpy="0 0 0"/>
     </joint>
     <link name="${prefix}ensenso">
@@ -115,9 +120,9 @@
         <origin xyz="${chuck_tcp_x} ${chuck_tcp_y} ${chuck_tcp_z}" rpy="0 -${half_pi} 0"/>
     </joint>
-    <joint name="${prefix}chuck_to_blend_tcp_frame" type="fixed">
+    <!--joint name="${prefix}chuck_to_blend_tcp_frame" type="fixed">
         <parent link="${prefix}chuck_tip_frame"/>
         <child link="${prefix}tcp_frame"/>
         <origin xyz="${blend_tcp_x} ${blend_tcp_y} ${blend_tcp_z}" rpy="0 0 0"/>
-    </joint>
+    </joint-->
     <!--Frames for the keyence profilometer-->
     <link name="${prefix}keyence_sensor_optical_frame"/>  <!--The emitter lens-->
